Commit message: Обновлены параметры планирования и добавлены новые файлы для модуля планирования движения, включая C++ и Python реализации.

File: src/iiwa_description/urdf/joints.xacro (robot description, xacro)
@@ -10,29 +10,36 @@
     <xacro:revolute_joint jname="joint1" parent="base_link" child="link1"
                         xyz="0 0 0.3375" rpy="0 0 0" axis="0 0 -1"
-                        lower="-2.97" upper="2.97" effort="500" velocity="1.71"/>
+                        lower="-2.97" upper="2.97" effort="500"
+                        velocity="1.71" damping="0.5"/>
     <!-- joint2 -->
     <xacro:revolute_joint jname="joint2" parent="link1" child="link2"
                         xyz="0 0 0" rpy="-1.5708 0 0" axis="0 0 1"
-                        lower="-2.09" upper="2.09" effort="500" velocity="1.71"/>
+                        lower="-2.09" upper="2.09" effort="500"
+                        velocity="1.71" damping="0.5"/>
     <!-- joint3 -->
     <xacro:revolute_joint jname="joint3" parent="link2" child="link3"
                         xyz="0 -0.3993 0" rpy="1.5708 0 0" axis="0 0 -1"
-                        lower="-2.97" upper="2.97" effort="500" velocity="1.75"/>
+                        lower="-2.97" upper="2.97" effort="500"
+                        velocity="1.75" damping="0.5"/>
     <!-- joint4 -->
     <xacro:revolute_joint jname="joint4" parent="link3" child="link4"
                         xyz="0 0 0" rpy="-1.5708 0 0" axis="0 0 -1"
-                        lower="-2.09" upper="2.09" effort="500" velocity="2.27"/>
+                        lower="-2.09" upper="2.09" effort="500"
+                        velocity="2.27" damping="0.5"/>
     <!-- joint5 -->
     <xacro:revolute_joint jname="joint5" parent="link4" child="link5"
                         xyz="0 -0.3993 0" rpy="1.5708 0 0" axis="0 0 -1"
-                        lower="-2.97" upper="2.97" effort="500" velocity="2.44"/>
+                        lower="-2.97" upper="2.97" effort="500"
+                        velocity="2.44" damping="0.5"/>
     <!-- joint6 -->
     <xacro:revolute_joint jname="joint6" parent="link5" child="link6"
                         xyz="0 0 0" rpy="-1.5708 0 0" axis="0 0 1"
-                        lower="-2.09" upper="2.09" effort="500" velocity="3.14"/>
+                        lower="-2.09" upper="2.09" effort="500"
+                        velocity="3.14" damping="0.5"/>
     <!-- joint7 -->
     <xacro:revolute_joint jname="joint7" parent="link6" child="link7"
                         xyz="0 -0.126 0" rpy="1.5708 0 0" axis="0 0 1"
-                        lower="-3.05" upper="3.05" effort="500" velocity="3.14"/>
+                        lower="-3.05" upper="3.05" effort="500"
+                        velocity="3.14" damping="0.5"/>
     <joint name="tools_joint" type="fixed">
         <origin xyz="0.0 0.0 0.0" rpy="0.0 0.0 0.0"/>

File: src/iiwa_description/urdf/macros.xacro (robot description, xacro)
@@ -27,5 +27,5 @@
     </xacro:macro>
     <!-- Макрос для описания соединений -->
-    <xacro:macro name="revolute_joint" params="jname parent child xyz rpy axis lower upper effort velocity">
+    <xacro:macro name="revolute_joint" params="jname parent child xyz rpy axis lower upper effort velocity damping">
         <joint name="${jname}" type="revolute">
             <origin xyz="${xyz}" rpy="${rpy}"/>
@@ -34,4 +34,5 @@
             <axis xyz="${axis}"/>
             <limit lower="${lower}" upper="${upper}" effort="${effort}" velocity="${velocity}"/>
+            <dynamics damping="${damping}"/>
         </joint>
     </xacro:macro>

File: src/iiwa_description/urdf/params.xacro (robot description, xacro)
@@ -2,12 +2,12 @@
 <robot xmlns:xacro="http://www.ros.org/wiki/xacro" xacro:version="1.0">
     <!-- Массы звеньев -->
-    <xacro:property name="mass_base" value="30.2763517543289"/>
-    <xacro:property name="mass_link1" value="21.1627406257303"/>
-    <xacro:property name="mass_link2" value="25.1403147192251"/>
-    <xacro:property name="mass_link3" value="21.1627874292289"/>
-    <xacro:property name="mass_link4" value="25.140328983289"/>
-    <xacro:property name="mass_link5" value="9.53466992761605"/>
-    <xacro:property name="mass_link6" value="14.2007599322815"/>
-    <xacro:property name="mass_link7" value="2.47156969383589"/>
+    <xacro:property name="mass_base" value="0.1"/>
+    <xacro:property name="mass_link1" value="4"/>
+    <xacro:property name="mass_link2" value="4"/>
+    <xacro:property name="mass_link3" value="3"/>
+    <xacro:property name="mass_link4" value="2.7"/>
+    <xacro:property name="mass_link5" value="1.7"/>
+    <xacro:property name="mass_link6" value="1.8"/>
+    <xacro:property name="mass_link7" value="0.3"/>
     <!-- Общие цвета / материал -->
     <xacro:property name="color_r" value="0.647058823529412"/>
