Commit message: Add gripper model and configuration for iiwa7 robot
- Created URDF model for gripper including links and joints.
- Added XACRO files for gripper components: gripper.xacro, gripper_links.xacro, gripper_joints.xacro, gripper_macros.xacro, and gripper_meshes.xacro.
- Integrated gripper into iiwa7 digital twin configuration.
- Defined properties and macros for gripper components to facilitate easier modifications and reuse.

File: src/iiwa_description/urdf/iiwa7_digital.urdf.xacro (robot description, xacro)
@@ -10,4 +10,5 @@
     <xacro:include filename="$(find iiwa_description)/urdf/links.xacro"/>
     <xacro:include filename="$(find iiwa_description)/urdf/joints.xacro"/>
+    <xacro:include filename="$(find iiwa_description)/urdf/gripper/gripper.xacro"/>
     <webots>
         <plugin type="webots_ros2_control::Ros2Control"/>
@@ -122,4 +123,12 @@
             <state_interface name="effort"/>
         </joint>
+        <!-- Захват -->
+        <!-- <joint name="base_screw">
+            <command_interface name="position"/>
+            <state_interface name="position">
+                <param name="initial_value">0.0</param>
+            </state_interface>
+            <state_interface name="velocity"/>
+        </joint> -->
     </ros2_control>
 </robot>

File: src/iiwa_description/urdf/iiwa7_fri.urdf.xacro (robot description, xacro)
@@ -13,4 +13,5 @@
     <xacro:include filename="$(find iiwa_description)/urdf/links.xacro"/>
     <xacro:include filename="$(find iiwa_description)/urdf/joints.xacro"/>
+    <xacro:include filename="$(find iiwa_description)/urdf/gripper/gripper.xacro"/>
     <ros2_control name="iiwaFRIControl" type="system">
         <hardware>

Commit message: Refactor launch files and update robot description for iiwa7 configuration

File: src/iiwa_description/urdf/iiwa7_digital.urdf.xacro (robot description, xacro)
@@ -4,9 +4,4 @@
     <xacro:arg name="initial_positions_file"
                default="$(find iiwa_config)/config/moveit/initial_positions.yaml"/>
-    <xacro:arg name="simulate" default="false"/>
-    <!-- Аргументы только для реального робота -->
-    <xacro:arg name="robot_ip" default="192.170.10.2"/>
-    <xacro:arg name="fri_port" default="30200"/>
-    <xacro:arg name="command_mode" default="position"/>
     <xacro:property name="initial_positions"
                     value="${xacro.load_yaml('$(arg initial_positions_file)')['initial_positions']}"/>
@@ -16,34 +11,11 @@
     <xacro:include filename="$(find iiwa_description)/urdf/joints.xacro"/>
     <xacro:include filename="$(find iiwa_description)/urdf/gripper/gripper.xacro"/>
-    <xacro:if value="$(arg simulate)">
-        <gazebo>
-            <plugin filename="gz_ros2_control-system"
-                    name="gz_ros2_control::GazeboSimROS2ControlPlugin">
-                <parameters>$(find iiwa_config)/config/moveit/iiwa_controller.yaml</parameters>
-                <ros>
-                    <remapping>~/robot_description:=/robot_description</remapping>
-                </ros>
-            </plugin>
-        </gazebo>
-    </xacro:if>
-    <!-- <webots>
+    <webots>
         <plugin type="webots_ros2_control::Ros2Control"/>
-    </webots> -->
-    <ros2_control name="iiwaControl" type="system">
-        <xacro:if value="$(arg simulate)">
-            <hardware>
-                <plugin>gz_ros2_control/GazeboSimSystem</plugin>
-            </hardware>
-        </xacro:if>
-        <hardware>
-            <plugin>iiwa_controller/IIWAHardwareInterface</plugin>
-            <param name="robot_ip">$(arg robot_ip)</param>
-            <param name="fri_port">$(arg fri_port)</param>
-            <param name="simulate">$(arg simulate)</param>
-            <param name="command_mode">$(arg command_mode)</param>
+    </webots>
+    <ros2_control name="iiwaGazeboControl" type="system">
+         <hardware>
+            <plugin>webots_ros2_control::Ros2ControlSystem</plugin>
         </hardware>
-         <!-- <hardware>
-            <plugin>webots_ros2_control::Ros2ControlSystem</plugin>
-        </hardware> -->
         <joint name="joint1">
             <command_interface name="position">
@@ -123,11 +95,4 @@
             <state_interface name="effort"/>
         </joint>
-        <joint name="base_screw">
-            <command_interface name="position"/>
-            <state_interface name="position">
-                <param name="initial_value">0.0</param>
-            </state_interface>
-            <state_interface name="velocity"/>
-        </joint>
     </ros2_control>
 </robot>
