Commit message: Реализован спавн робота с контроллерами в виртуальной среде `webots`

File: src/iiwa_description/urdf/iiwa7.urdf.xacro (robot description, xacro)
@@ -5,3 +5,39 @@
     <xacro:include filename="$(find iiwa_description)/urdf/links.xacro"/>
     <xacro:include filename="$(find iiwa_description)/urdf/joints.xacro"/>
+    <webots>
+        <plugin type="webots_ros2_control::Ros2Control"/>
+    </webots>
+    <ros2_control name="iiwaWebotsControl" type="system">
+        <hardware>
+            <plugin>webots_ros2_control::Ros2ControlSystem</plugin>
+        </hardware>
+        <joint name="joint1">
+            <state_interface name="position"/>
+            <command_interface name="position"/>
+        </joint>
+        <joint name="joint2">
+            <state_interface name="position"/>
+            <command_interface name="position"/>
+        </joint>
+        <joint name="joint3">
+            <state_interface name="position"/>
+            <command_interface name="position"/>
+        </joint>
+        <joint name="joint4">
+            <state_interface name="position"/>
+            <command_interface name="position"/>
+        </joint>
+        <joint name="joint5">
+            <state_interface name="position"/>
+            <command_interface name="position"/>
+        </joint>
+        <joint name="joint6">
+            <state_interface name="position"/>
+            <command_interface name="position"/>
+        </joint>
+        <joint name="joint7">
+            <state_interface name="position"/>
+            <command_interface name="position"/>
+        </joint>
+    </ros2_control>
 </robot>

File: src/iiwa_description/urdf/joints.xacro (robot description, xacro)
@@ -10,33 +10,33 @@
     <xacro:revolute_joint jname="joint1" parent="base_link" child="link1"
                         xyz="0 0 0.3375" rpy="0 0 0" axis="0 0 -1"
-                        lower="-2.97" upper="2.97" effort="176" velocity="1.71"/>
+                        lower="-2.97" upper="2.97" effort="500" velocity="1.71"/>
     <!-- joint2 -->
     <xacro:revolute_joint jname="joint2" parent="link1" child="link2"
                         xyz="0 0 0" rpy="-1.5708 0 0" axis="0 0 1"
-                        lower="-2.09" upper="2.09" effort="176" velocity="1.71"/>
+                        lower="-2.09" upper="2.09" effort="500" velocity="1.71"/>
     <!-- joint3 -->
     <xacro:revolute_joint jname="joint3" parent="link2" child="link3"
                         xyz="0 -0.3993 0" rpy="1.5708 0 0" axis="0 0 -1"
-                        lower="-2.97" upper="2.97" effort="110" velocity="1.75"/>
+                        lower="-2.97" upper="2.97" effort="500" velocity="1.75"/>
     <!-- joint4 -->
     <xacro:revolute_joint jname="joint4" parent="link3" child="link4"
                         xyz="0 0 0" rpy="-1.5708 0 0" axis="0 0 -1"
-                        lower="-2.09" upper="2.09" effort="110" velocity="2.27"/>
+                        lower="-2.09" upper="2.09" effort="500" velocity="2.27"/>
     <!-- joint5 -->
     <xacro:revolute_joint jname="joint5" parent="link4" child="link5"
                         xyz="0 -0.3993 0" rpy="1.5708 0 0" axis="0 0 -1"
-                        lower="-2.97" upper="2.97" effort="110" velocity="2.44"/>
+                        lower="-2.97" upper="2.97" effort="500" velocity="2.44"/>
     <!-- joint6 -->
     <xacro:revolute_joint jname="joint6" parent="link5" child="link6"
                         xyz="0 0 0" rpy="-1.5708 0 0" axis="0 0 1"
-                        lower="-2.09" upper="2.09" effort="40" velocity="3.14"/>
+                        lower="-2.09" upper="2.09" effort="500" velocity="3.14"/>
     <!-- joint7 -->
     <xacro:revolute_joint jname="joint7" parent="link6" child="link7"
                         xyz="0 -0.126 0" rpy="1.5708 0 0" axis="0 0 1"
-                        lower="-3.05" upper="3.05" effort="40" velocity="3.14"/>
+                        lower="-3.05" upper="3.05" effort="500" velocity="3.14"/>
     <joint name="tools_joint" type="fixed">
         <origin xyz="0.0 0.0 0.0" rpy="0.0 0.0 0.0"/>
         <parent link="link7"/>
-        <child link="link7_ee"/>
+        <child link="link_ee"/>
     </joint>
 </robot>

File: src/iiwa_description/urdf/links.xacro (robot description, xacro)
@@ -90,4 +90,4 @@
                      mesh_vision="${mesh_link7_v}"
                      mesh_collision="${mesh_link7_c}"/>
-    <link name="link7_ee" />
+    <link name="link_ee" />
 </robot>

File: src/iiwa_description/urdf/meshes.xacro (robot description, xacro)
@@ -1,5 +1,5 @@
 <?xml version="1.0"?>
 <robot xmlns:xacro="http://www.ros.org/wiki/xacro" xacro:version="1.0">
-    <xacro:property name="pkg" value="package://iiwa_description/meshes"/>
+    <xacro:property name="pkg" value="package://iiwa_description/resource/meshes"/>
     <!-- Меши отображения -->
     <xacro:property name="mesh_base_v" value="${pkg}/visual/base_link.DAE"/>

Commit message: добавлена поддержка moveit

File: src/iiwa_description/urdf/iiwa7.urdf.xacro (robot description, xacro)
@@ -1,4 +1,9 @@
 <?xml version="1.0"?>
 <robot xmlns:xacro="http://www.ros.org/wiki/xacro" name="iiwa7">
+    <!-- Аргукменты -->
+    <xacro:arg name="initial_positions_file"
+           default="$(find iiwa_bringup)/config/initial_positions.yaml"/>
+    <xacro:property name="initial_positions"
+                value="${xacro.load_yaml('$(arg initial_positions_file)')['initial_positions']}"/>
     <xacro:include filename="$(find iiwa_description)/urdf/params.xacro"/>
     <xacro:include filename="$(find iiwa_description)/urdf/macros.xacro"/>
@@ -11,32 +16,47 @@
         <hardware>
             <plugin>webots_ros2_control::Ros2ControlSystem</plugin>
+            <!-- <plugin>mock_components/GenericSystem</plugin> -->
         </hardware>
-        <joint name="joint1">
-            <state_interface name="position"/>
+       <joint name="joint1">
             <command_interface name="position"/>
+            <state_interface name="position">
+                <param name="initial_value">${initial_positions['joint1']}</param>
+            </state_interface>
         </joint>
         <joint name="joint2">
-            <state_interface name="position"/>
             <command_interface name="position"/>
+            <state_interface name="position">
+                <param name="initial_value">${initial_positions['joint2']}</param>
+            </state_interface>
         </joint>
         <joint name="joint3">
-            <state_interface name="position"/>
             <command_interface name="position"/>
+            <state_interface name="position">
+                <param name="initial_value">${initial_positions['joint3']}</param>
+            </state_interface>
         </joint>
         <joint name="joint4">
-            <state_interface name="position"/>
             <command_interface name="position"/>
+            <state_interface name="position">
+                <param name="initial_value">${initial_positions['joint4']}</param>
+            </state_interface>
         </joint>
         <joint name="joint5">
-            <state_interface name="position"/>
             <command_interface name="position"/>
+            <state_interface name="position">
+                <param name="initial_value">${initial_positions['joint5']}</param>
+            </state_interface>
         </joint>
         <joint name="joint6">
-            <state_interface name="position"/>
             <command_interface name="position"/>
+            <state_interface name="position">
+                <param name="initial_value">${initial_positions['joint6']}</param>
+            </state_interface>
         </joint>
         <joint name="joint7">
-            <state_interface name="position"/>
             <command_interface name="position"/>
+            <state_interface name="position">
+                <param name="initial_value">${initial_positions['joint7']}</param>
+            </state_interface>
         </joint>
     </ros2_control>

Commit message: Add URDF and XACRO files for iiwa7 robot and tool patron
- Created iiwa7_gazebo.urdf to define the iiwa7 robot model with detailed links, joints, and Gazebo integration.
- Introduced patron.xacro for the tool patron, including its inertial properties, visual representation, and collision geometry.

File: src/iiwa_description/urdf/iiwa7.urdf.xacro (robot description, xacro)
@@ -13,5 +13,6 @@
     <xacro:include filename="$(find iiwa_description)/urdf/links.xacro"/>
     <xacro:include filename="$(find iiwa_description)/urdf/joints.xacro"/>
-    <xacro:include filename="$(find iiwa_description)/urdf/gripper/gripper.xacro"/>
+    <!-- <xacro:include filename="$(find iiwa_description)/urdf/gripper/gripper.xacro"/> -->
+    <xacro:include filename="$(find iiwa_description)/urdf/tools/patron.xacro"/>
     <xacro:if value="$(arg simulate)">
         <gazebo>
@@ -105,11 +106,4 @@
                 <state_interface name="effort"/>
             </joint>
-            <joint name="base_screw">
-                <command_interface name="position"/>
-                <state_interface name="position">
-                    <param name="initial_value">0.0</param>
-                </state_interface>
-                <state_interface name="velocity"/>
-            </joint>
         </ros2_control>
     </xacro:if>

File: src/iiwa_description/urdf/iiwa7_digital.urdf.xacro (robot description, xacro)
@@ -10,5 +10,6 @@
     <xacro:include filename="$(find iiwa_description)/urdf/links.xacro"/>
     <xacro:include filename="$(find iiwa_description)/urdf/joints.xacro"/>
-    <xacro:include filename="$(find iiwa_description)/urdf/gripper/gripper.xacro"/>
+    <!-- <xacro:include filename="$(find iiwa_description)/urdf/gripper/gripper.xacro"/> -->
+    <xacro:include filename="$(find iiwa_description)/urdf/tools/patron.xacro"/>
     <webots>
         <plugin type="webots_ros2_control::Ros2Control"/>

File: src/iiwa_description/urdf/meshes.xacro (robot description, xacro)
@@ -3,20 +3,20 @@
     <xacro:property name="pkg" value="package://iiwa_description/resource/meshes"/>
     <!-- Меши отображения -->
-    <xacro:property name="mesh_base_v" value="${pkg}/visual/base_link.DAE"/>
-    <xacro:property name="mesh_link1_v" value="${pkg}/visual/link1.DAE"/>
-    <xacro:property name="mesh_link2_v" value="${pkg}/visual/link2.DAE"/>
-    <xacro:property name="mesh_link3_v" value="${pkg}/visual/link3.DAE"/>
-    <xacro:property name="mesh_link4_v" value="${pkg}/visual/link4.DAE"/>
-    <xacro:property name="mesh_link5_v" value="${pkg}/visual/link5.DAE"/>
-    <xacro:property name="mesh_link6_v" value="${pkg}/visual/link6.DAE"/>
-    <xacro:property name="mesh_link7_v" value="${pkg}/visual/link7.DAE"/>
+    <xacro:property name="mesh_base_v" value="${pkg}/iiwa/visual/base_link.DAE"/>
+    <xacro:property name="mesh_link1_v" value="${pkg}/iiwa/visual/link1.DAE"/>
+    <xacro:property name="mesh_link2_v" value="${pkg}/iiwa/visual/link2.DAE"/>
+    <xacro:property name="mesh_link3_v" value="${pkg}/iiwa/visual/link3.DAE"/>
+    <xacro:property name="mesh_link4_v" value="${pkg}/iiwa/visual/link4.DAE"/>
+    <xacro:property name="mesh_link5_v" value="${pkg}/iiwa/visual/link5.DAE"/>
+    <xacro:property name="mesh_link6_v" value="${pkg}/iiwa/visual/link6.DAE"/>
+    <xacro:property name="mesh_link7_v" value="${pkg}/iiwa/visual/link7.DAE"/>
     <!-- Меши колизии -->
-    <xacro:property name="mesh_base_c" value="${pkg}/collision/base_link.STL"/>
-    <xacro:property name="mesh_link1_c" value="${pkg}/collision/link1.STL"/>
-    <xacro:property name="mesh_link2_c" value="${pkg}/collision/link2.STL"/>
-    <xacro:property name="mesh_link3_c" value="${pkg}/collision/link3.STL"/>
-    <xacro:property name="mesh_link4_c" value="${pkg}/collision/link4.STL"/>
-    <xacro:property name="mesh_link5_c" value="${pkg}/collision/link5.STL"/>
-    <xacro:property name="mesh_link6_c" value="${pkg}/collision/link6.STL"/>
-    <xacro:property name="mesh_link7_c" value="${pkg}/collision/link7.STL"/>
+    <xacro:property name="mesh_base_c" value="${pkg}/iiwa/collision/base_link.STL"/>
+    <xacro:property name="mesh_link1_c" value="${pkg}/iiwa/collision/link1.STL"/>
+    <xacro:property name="mesh_link2_c" value="${pkg}/iiwa/collision/link2.STL"/>
+    <xacro:property name="mesh_link3_c" value="${pkg}/iiwa/collision/link3.STL"/>
+    <xacro:property name="mesh_link4_c" value="${pkg}/iiwa/collision/link4.STL"/>
+    <xacro:property name="mesh_link5_c" value="${pkg}/iiwa/collision/link5.STL"/>
+    <xacro:property name="mesh_link6_c" value="${pkg}/iiwa/collision/link6.STL"/>
+    <xacro:property name="mesh_link7_c" value="${pkg}/iiwa/collision/link7.STL"/>
 </robot>

Commit message: Add cameraD455 mesh file to iiwa_description resources

File: src/iiwa_description/urdf/iiwa7.urdf.xacro (robot description, xacro)
@@ -17,4 +17,20 @@
         <webots>
             <plugin type="webots_ros2_control::Ros2Control"/>
+            <device reference="camera_rgb" type="Camera">
+                <ros>
+                    <topicName>/camera/color</topicName>
+                    <updateRate>30</updateRate>
+                    <alwaysOn>True</alwaysOn>
+                    <frameName>camera_optical_frame</frameName>
+                </ros>
+            </device>
+            <device reference="camera_depth" type="RangeFinder">
+                <ros>
+                    <topicName>/camera/depth</topicName>
+                    <updateRate>30</updateRate>
+                    <alwaysOn>True</alwaysOn>
+                    <frameName>camera_optical_frame</frameName>
+                </ros>
+            </device>
         </webots>
         <ros2_control name="iiwaGazeboControl" type="system">

File: src/iiwa_description/urdf/tools/patron.xacro (robot description, xacro)
@@ -1,21 +1,69 @@
 <?xml version="1.0"?>
 <robot xmlns:xacro="http://www.ros.org/wiki/xacro" name="tool_patron">
+    <link name="camera_holder">
+        <inertial>
+            <origin xyz="0.0 0.0 0.0" rpy="0.0 0.0 0.0"/>
+            <mass value="0.09"/>
+            <inertia ixx="0.0" ixy="0.0" ixz="0.0"
+                     iyy="0.0" iyz="0.0" izz="0.0"/>
+        </inertial>
+        <visual name="">
+            <origin xyz="0.0 0.0 0.0" rpy="0.0 0.0 0.0"/>
+            <geometry>
+                <!-- <mesh filename="/home/daniel/dev/kuka_iiwa7_ros2/src/iiwa_description/resource/meshes/tools/CameraHolder.dae" /> -->
+                <mesh filename="package://iiwa_description/resource/meshes/tools/CameraHolder.dae"/>
+            </geometry>
+        </visual>
+        <collision>
+            <origin xyz="0.0 0.0 0.015" rpy="0.0 0.0 0.0"/>
+            <geometry>
+                <cylinder radius="0.035" length="0.03"/>
+            </geometry>
+        </collision>
+        <collision>
+            <origin xyz="0.0 0.08 0.015" rpy="0.0 0.0 0.0"/>
+            <geometry>
+                <box size="0.03 0.1 0.03"/>
+            </geometry>
+        </collision>
+    </link>
+    <link name="camera_hand">
+        <inertial>
+            <origin xyz="0.0 0.0 0.0" rpy="0.0 0.0 0.0"/>
+            <mass value="0.0"/>
+            <inertia ixx="0.0" ixy="0.0" ixz="0.0" iyy="0.0" iyz="0.0" izz="0.0"/>
+        </inertial>
+        <visual>
+            <origin xyz="-0.06 0.0 0.0" rpy="0.0 0.0 0.0"/>
+            <geometry>
+                <!-- <mesh filename="/home/daniel/dev/kuka_iiwa7_ros2/src/iiwa_description/resource/meshes/tools/cameraD455.dae" /> -->
+                <mesh filename="package://iiwa_description/resource/meshes/tools/cameraD455.dae"/>
+            </geometry>
+        </visual>
+        <collision>
+            <origin xyz="0.0 0.014 0.0125" rpy="0.0 0.0 0.0"/>
+            <geometry>
+                <box size="0.12 0.025 0.025"/>
+            </geometry>
+        </collision>
+    </link>
     <link name="patron">
         <inertial>
             <origin xyz="0.0 0.0 0.0" rpy="0.0 0.0 0.0"/>
-            <mass value="0.69"/>
-            <inertia ixx="0.000483150" ixy="0.0" ixz="0.0"
-                     iyy="0.000483150" iyz="0.0" izz="0.000241750"/>
+            <mass value="0.03"/>
+            <inertia ixx="0.0" ixy="0.0" ixz="0.0"
+            iyy="0.0" iyz="0.0" izz="0.0"/>
         </inertial>
-        <visual>
+        <visual name="">
             <origin xyz="0.0 0.0 0.0" rpy="0.0 0.0 0.0"/>
             <geometry>
+                <!-- <mesh filename="/home/daniel/dev/kuka_iiwa7_ros2/src/iiwa_description/resource/meshes/tools/patron.dae" /> -->
                 <mesh filename="package://iiwa_description/resource/meshes/tools/patron.dae"/>
             </geometry>
         </visual>
         <collision>
-            <origin xyz="0.0 0.0 0.0354" rpy="0.0 0.0 0.0"/>
+            <origin xyz="0.0 0.0 0.027" rpy="0.0 0.0 0.0"/>
             <geometry>
-                <cylinder radius="0.0315" length="0.071"/>
+                <cylinder radius="0.021" length="0.055"/>
             </geometry>
         </collision>
@@ -23,6 +71,64 @@
     <joint name="tool" type="fixed">
         <parent link="link_ee"/>
+        <child link="camera_holder"/>
+        <origin xyz="0 0 0" rpy="0 0 1.5708"/>
+    </joint>
+    <joint name="cameraHolder_patron" type="fixed">
+        <origin xyz="0.0 0.0 0.03" rpy="0.0 0.0 0.0"/>
+        <parent link="camera_holder"/>
         <child link="patron"/>
-        <origin xyz="0 0 0" rpy="0 0 0"/>
     </joint>
+    <joint name="cameraHolder_cameraD455" type="fixed">
+        <origin xyz="0.0 0.1 0.014" rpy="0.0 0.0 0.0"/>
+        <parent link="camera_holder"/>
+        <child link="camera_hand"/>
+    </joint>
+    <link name="camera_optical_frame"/>
+    <joint name="camera_hand_to_optical" type="fixed">
+        <origin xyz="0.0 0.0 0.0" rpy="0.0 0.0 3.14159"/>
+        <parent link="camera_hand"/>
+        <child link="camera_optical_frame"/>
+    </joint>
+    <gazebo reference="camera_optical_frame">
+        <sensor type="camera" name="camera_rgb">
+            <camera>
+                <horizontal_fov>1.5708</horizontal_fov>
+                <image>
+                    <width>640</width>
+                    <height>480</height>
+                    <format>R8G8B8</format>
+                </image>
+                <clip>
+                    <near>0.1</near>
+                    <far>10.0</far>
+                </clip>
+                <noise>
+                    <type>gaussian</type>
+                    <stddev>0.005</stddev>
+                </noise>
+            </camera>
+        </sensor>
+        <sensor type="depth" name="camera_depth">
+            <camera>
+                <horizontal_fov>1.5184</horizontal_fov>
+                <image>
+                    <width>640</width>
+                    <height>480</height>
+                </image>
+                <clip>
+                    <near>0.52</near>
+                    <far>6.0</far>
+                </clip>
+            </camera>
+            <range>
+                <min>0.52</min>
+                <max>6.0</max>
+                <resolution>0.001</resolution>
+            </range>
+            <noise>
+                <type>gaussian</type>
+                <stddev>0.02</stddev>
+            </noise>
+        </sensor>
+    </gazebo>
 </robot>
