Commit message: Refactor code structure for improved readability and maintainability

File: src/iiwa_description/urdf/iiwa7.urdf.xacro (robot description, xacro)
@@ -13,5 +13,5 @@
     <xacro:include filename="$(find iiwa_description)/urdf/links.xacro"/>
     <xacro:include filename="$(find iiwa_description)/urdf/joints.xacro"/>
-    <xacro:include filename="$(find iiwa_description)/urdf/tools/patron.xacro"/>
+    <xacro:include filename="$(find iiwa_description)/urdf/tools/patronv2.xacro"/>
     <xacro:if value="$(arg simulate)">
         <webots>
@@ -23,12 +23,4 @@
                     <alwaysOn>True</alwaysOn>
                     <frameName>camera_optical_frame</frameName>
-                </ros>
-            </device>
-            <device reference="example_camera" type="Camera">
-                <ros>
-                    <topicName>/camera_example/color</topicName>
-                    <updateRate>30</updateRate>
-                    <alwaysOn>True</alwaysOn>
-                    <frameName>example_camera</frameName>
                 </ros>
             </device>

File: src/iiwa_description/urdf/tools/patron.xacro (robot description, xacro)
@@ -4,13 +4,12 @@
         <inertial>
             <origin xyz="0.0 0.0 0.0" rpy="0.0 0.0 0.0"/>
-            <mass value="0.09"/>
-            <inertia ixx="0.0" ixy="0.0" ixz="0.0"
-                     iyy="0.0" iyz="0.0" izz="0.0"/>
+            <mass value="0.15"/>
+            <inertia ixx="0.000073" ixy="0.0" ixz="0.0"
+                     iyy="0.000136" iyz="0.0" izz="0.000186"/>
         </inertial>
         <visual name="">
             <origin xyz="0.0 0.0 0.0" rpy="0.0 0.0 0.0"/>
             <geometry>
-                <!-- <mesh filename="/home/daniel/dev/kuka_iiwa7_ros2/src/iiwa_description/resource/meshes/tools/CameraHolder.dae" /> -->
-                <mesh filename="package://iiwa_description/resource/meshes/tools/CameraHolder.dae"/>
+                <mesh filename="package://iiwa_description/resource/meshes/tools/CameraHolder.dae" />
             </geometry>
         </visual>
@@ -28,15 +27,55 @@
         </collision>
     </link>
+    <link name="patron">
+        <inertial>
+            <origin xyz="0.0 0.0 0.0" rpy="0.0 0.0 0.0"/>
+            <mass value="0.35"/>
+            <inertia ixx="0.000127" ixy="0.0" ixz="0.0"
+                     iyy="0.000127" iyz="0.0" izz="0.000077"/>
+        </inertial>
+        <visual name="">
+            <origin xyz="0.0 0.0 0.0" rpy="0.0 0.0 0.0"/>
+            <geometry>
+                <mesh filename="package://iiwa_description/resource/meshes/tools/patron.dae" />
+            </geometry>
+        </visual>
+        <collision>
+            <origin xyz="0.0 0.0 0.027" rpy="0.0 0.0 0.0"/>
+            <geometry>
+                <cylinder radius="0.021" length="0.055"/>
+            </geometry>
+        </collision>
+    </link>
+    <link name="camera_corner">
+        <inertial>
+            <origin xyz="0.0 0.0 0.0" rpy="0.0 0.0 0.0"/>
+            <mass value="0.1"/>
+            <inertia ixx="0.0000094" ixy="0.0" ixz="0.0"
+                     iyy="0.000131"  iyz="0.0" izz="0.000135"/>
+        </inertial>
+        <visual name="">
+            <origin xyz="0.0 0.0 0.0" rpy="0.0 0.0 0.0"/>
+            <geometry>
+                <mesh filename="package://iiwa_description/resource/meshes/tools/camera_corner.dae" />
+            </geometry>
+        </visual>
+        <collision>
+            <origin xyz="0 0.116 0.022" rpy="0.0 0.0 0.0"/>
+            <geometry>
+                <box size="0.124 0.029 0.017"/>
+            </geometry>
+        </collision>
+    </link>
     <link name="camera_hand">
         <inertial>
             <origin xyz="0.0 0.0 0.0" rpy="0.0 0.0 0.0"/>
-            <mass value="0.0"/>
-            <inertia ixx="0.0" ixy="0.0" ixz="0.0" iyy="0.0" iyz="0.0" izz="0.0"/>
+            <mass value="0.2"/>
+            <inertia ixx="0.000021" ixy="0.0" ixz="0.0"
+                     iyy="0.000250" iyz="0.0" izz="0.000250"/>
         </inertial>
         <visual>
             <origin xyz="-0.06 0.0 0.0" rpy="0.0 0.0 0.0"/>
             <geometry>
-                <!-- <mesh filename="/home/daniel/dev/kuka_iiwa7_ros2/src/iiwa_description/resource/meshes/tools/cameraD455.dae" /> -->
-                <mesh filename="package://iiwa_description/resource/meshes/tools/cameraD455.dae"/>
+                <mesh filename="package://iiwa_description/resource/meshes/tools/cameraD455.dae" />
             </geometry>
         </visual>
@@ -48,25 +87,5 @@
         </collision>
     </link>
-    <link name="patron">
-        <inertial>
-            <origin xyz="0.0 0.0 0.0" rpy="0.0 0.0 0.0"/>
-            <mass value="0.03"/>
-            <inertia ixx="0.0" ixy="0.0" ixz="0.0"
-            iyy="0.0" iyz="0.0" izz="0.0"/>
-        </inertial>
-        <visual name="">
-            <origin xyz="0.0 0.0 0.0" rpy="0.0 0.0 0.0"/>
-            <geometry>
-                <!-- <mesh filename="/home/daniel/dev/kuka_iiwa7_ros2/src/iiwa_description/resource/meshes/tools/patron.dae" /> -->
-                <mesh filename="package://iiwa_description/resource/meshes/tools/patron.dae"/>
-            </geometry>
-        </visual>
-        <collision>
-            <origin xyz="0.0 0.0 0.027" rpy="0.0 0.0 0.0"/>
-            <geometry>
-                <cylinder radius="0.021" length="0.055"/>
-            </geometry>
-        </collision>
-    </link>
+    <link name="camera_optical_frame"/>
     <joint name="tool" type="fixed">
         <parent link="link_ee"/>
@@ -74,17 +93,21 @@
         <origin xyz="0 0 0" rpy="0 0 1.5708"/>
     </joint>
-    <joint name="cameraHolder_patron" type="fixed">
-        <origin xyz="0.0 0.0 0.03" rpy="0.0 0.0 0.0"/>
+    <joint name="camera_holder_patron" type="fixed">
+        <origin xyz="0.0 0.0 0.032" rpy="0.0 0.0 0.0"/>
         <parent link="camera_holder"/>
         <child link="patron"/>
     </joint>
-    <joint name="cameraHolder_cameraD455" type="fixed">
-        <origin xyz="0.0 0.1 0.014" rpy="0.0 0.0 0.0"/>
+    <joint name="camera_holder_corner" type="fixed">
+        <origin xyz="0.0 0.0 0.0" rpy="0.0 0.0 0.0"/>
         <parent link="camera_holder"/>
+        <child link="camera_corner"/>
+    </joint>
+    <joint name="camera_corner_camera" type="fixed">
+        <origin xyz="0.0 0.1 0.014" rpy="0.61 0.0 0.0"/>
+        <parent link="camera_corner"/>
         <child link="camera_hand"/>
     </joint>
-    <link name="camera_optical_frame"/>
     <joint name="camera_hand_to_optical" type="fixed">
-        <origin xyz="0.0 0.0 0.0" rpy="0.0 0.0 3.14159"/>
+        <origin xyz="0.0 0.0 0.0" rpy="0.0 0.0 0.0"/>
         <parent link="camera_hand"/>
         <child link="camera_optical_frame"/>
@@ -93,5 +116,5 @@
         <sensor type="camera" name="camera_rgb">
             <camera>
-                <horizontal_fov>1.5708</horizontal_fov>
+                <horizontal_fov>1.3089969</horizontal_fov>
                 <image>
                     <width>640</width>
@@ -111,5 +134,5 @@
         <sensor type="depth" name="camera_depth">
             <camera>
-                <horizontal_fov>1.5184</horizontal_fov>
+                <horizontal_fov>1.3089969</horizontal_fov>
                 <image>
                     <width>640</width>

Commit message: Refactor iiwa_controller_v2: Remove obsolete files and update URDF parameters
- Deleted `system_interface_type_values.hpp`, `package.xml`, `fri_client.cpp`, and `system_interface.cpp` as part of the cleanup process.
- Updated `iiwa7.urdf.xacro` to remove deprecated parameters and adjust command interface settings.
- Modified joint definitions in `joints.xacro` to include new friction and soft limit parameters.
- Enhanced `macros.xacro` to support additional joint properties for friction and safety control.
- Adjusted mass properties in `params.xacro` to reflect accurate values for the robot's components.

File: src/iiwa_description/urdf/iiwa7.urdf.xacro (robot description, xacro)
@@ -8,7 +8,4 @@
     <xacro:arg name="command_mode" default="position"/>
     <xacro:arg name="joint_position_tau" default="0.04"/>
-    <!-- iiwa_controller_v2: новые параметры. Убери эти строки при откате на v1 -->
-    <!-- <xacro:arg name="open_loop" default="true"/>
-    <xacro:arg name="rt_prio" default="80"/> -->
     <xacro:property name="initial_positions"
                     value="${xacro.load_yaml('$(arg initial_positions_file)')['initial_positions']}"/>
@@ -124,27 +121,4 @@
         <ros2_control name="iiwaFRIControl" type="system">
             <hardware>
-                <!-- ════════════════════════════════════════════════════════
-                     АКТИВНЫЙ ПЛАГИН: iiwa_controller_v2
-                     Чтобы вернуть v1 — раскомментируй блок v1 ниже
-                     и закомментируй блок v2.
-                     ════════════════════════════════════════════════════════ -->
-                <!-- ── v2 (активен) ──────────────────────────────────────── -->
-                <!-- <plugin>iiwa_controller_v2/SystemInterface</plugin> -->
-                <!-- <param name="robot_ip">$(arg robot_ip)</param> -->
-                <!-- <param name="fri_port">$(arg fri_port)</param> -->
-                <!-- <param name="simulate">false</param> -->
-                <!-- <param name="command_mode">$(arg command_mode)</param> -->
-                <!-- <param name="joint_position_tau">$(arg joint_position_tau)</param> -->
-                <!-- новые параметры v2: -->
-                <!-- <param name="open_loop">$(arg open_loop)</param> -->
-                <!-- <param name="rt_prio">$(arg rt_prio)</param> -->
-                <!-- ── v1 (закомментировано) ─────────────────────────────
-                <plugin>iiwa_controller/IIWAHardwareInterface</plugin>
-                <param name="robot_ip">$(arg robot_ip)</param>
-                <param name="fri_port">$(arg fri_port)</param>
-                <param name="simulate">false</param>
-                <param name="command_mode">$(arg command_mode)</param>
-                <param name="joint_position_tau">$(arg joint_position_tau)</param>
-                ─────────────────────────────────────────────────────────── -->
                 <plugin>iiwa_controller/IIWAHardwareInterface</plugin>
                 <param name="robot_ip">$(arg robot_ip)</param>
@@ -160,6 +134,6 @@
                 </command_interface>
                 <command_interface name="effort">
-                    <param name="min">-320</param>
-                    <param name="max"> 320</param>
+                    <param name="min">-200</param>
+                    <param name="max"> 200</param>
                 </command_interface>
                 <state_interface name="position">
@@ -175,6 +149,6 @@
                 </command_interface>
                 <command_interface name="effort">
-                    <param name="min">-320</param>
-                    <param name="max"> 320</param>
+                    <param name="min">-200</param>
+                    <param name="max"> 200</param>
                 </command_interface>
                 <state_interface name="position">
@@ -190,6 +164,6 @@
                 </command_interface>
                 <command_interface name="effort">
-                    <param name="min">-320</param>
-                    <param name="max"> 320</param>
+                    <param name="min">-200</param>
+                    <param name="max"> 200</param>
                 </command_interface>
                 <state_interface name="position">
@@ -205,6 +179,6 @@
                 </command_interface>
                 <command_interface name="effort">
-                    <param name="min">-320</param>
-                    <param name="max"> 320</param>
+                    <param name="min">-200</param>
+                    <param name="max"> 200</param>
                 </command_interface>
                 <state_interface name="position">
@@ -220,6 +194,6 @@
                 </command_interface>
                 <command_interface name="effort">
-                    <param name="min">-320</param>
-                    <param name="max"> 320</param>
+                    <param name="min">-200</param>
+                    <param name="max"> 200</param>
                 </command_interface>
                 <state_interface name="position">
@@ -235,6 +209,6 @@
                 </command_interface>
                 <command_interface name="effort">
-                    <param name="min">-320</param>
-                    <param name="max"> 320</param>
+                    <param name="min">-200</param>
+                    <param name="max"> 200</param>
                 </command_interface>
                 <state_interface name="position">
@@ -250,6 +224,6 @@
                 </command_interface>
                 <command_interface name="effort">
-                    <param name="min">-320</param>
-                    <param name="max"> 320</param>
+                    <param name="min">-200</param>
+                    <param name="max"> 200</param>
                 </command_interface>
                 <state_interface name="position">

File: src/iiwa_description/urdf/joints.xacro (robot description, xacro)
@@ -7,39 +7,46 @@
         <child link="base_link"/>
     </joint>
-    <!-- joint1 -->
+    <!-- joint1: ±170° hard, ±165° soft, k_velocity=10 -->
     <xacro:revolute_joint jname="joint1" parent="base_link" child="link1"
-                        xyz="0 0 0.3375" rpy="0 0 0" axis="0 0 -1"
-                        lower="-2.97" upper="2.97" effort="500"
-                        velocity="1.71" damping="0.5"/>
-    <!-- joint2 -->
+                        xyz="0 0 0.3375" rpy="0 0 0" axis="0 0 1"
+                        lower="-2.97" upper="2.97" effort="200"
+                        velocity="1.71" damping="10.0" friction="0.1"
+                        soft_lower="-2.8827" soft_upper="2.8827" k_velocity="10"/>
+    <!-- joint2: ±119° hard, ±114° soft -->
     <xacro:revolute_joint jname="joint2" parent="link1" child="link2"
                         xyz="0 0 0" rpy="-1.5708 0 0" axis="0 0 1"
-                        lower="-2.09" upper="2.09" effort="500"
-                        velocity="1.71" damping="0.5"/>
-    <!-- joint3 -->
+                        lower="-2.09" upper="2.09" effort="200"
+                        velocity="1.71" damping="10.0" friction="0.1"
+                        soft_lower="-2.0027" soft_upper="2.0027" k_velocity="10"/>
+    <!-- joint3: ±170° hard, ±165° soft -->
     <xacro:revolute_joint jname="joint3" parent="link2" child="link3"
                         xyz="0 -0.3993 0" rpy="1.5708 0 0" axis="0 0 -1"
-                        lower="-2.97" upper="2.97" effort="500"
-                        velocity="1.75" damping="0.5"/>
-    <!-- joint4 -->
+                        lower="-2.97" upper="2.97" effort="200"
+                        velocity="1.75" damping="10.0" friction="0.1"
+                        soft_lower="-2.8827" soft_upper="2.8827" k_velocity="10"/>
+    <!-- joint4: ±119° hard, ±114° soft -->
     <xacro:revolute_joint jname="joint4" parent="link3" child="link4"
                         xyz="0 0 0" rpy="-1.5708 0 0" axis="0 0 -1"
-                        lower="-2.09" upper="2.09" effort="500"
-                        velocity="2.27" damping="0.5"/>
-    <!-- joint5 -->
+                        lower="-2.09" upper="2.09" effort="200"
+                        velocity="2.27" damping="10.0" friction="0.1"
+                        soft_lower="-2.0027" soft_upper="2.0027" k_velocity="10"/>
+    <!-- joint5: ±170° hard, ±165° soft -->
     <xacro:revolute_joint jname="joint5" parent="link4" child="link5"
                         xyz="0 -0.3993 0" rpy="1.5708 0 0" axis="0 0 -1"
-                        lower="-2.97" upper="2.97" effort="500"
-                        velocity="2.44" damping="0.5"/>
-    <!-- joint6 -->
+                        lower="-2.97" upper="2.97" effort="200"
+                        velocity="2.44" damping="10.0" friction="0.1"
+                        soft_lower="-2.8827" soft_upper="2.8827" k_velocity="10"/>
+    <!-- joint6: ±119° hard, ±114° soft -->
     <xacro:revolute_joint jname="joint6" parent="link5" child="link6"
                         xyz="0 0 0" rpy="-1.5708 0 0" axis="0 0 1"
-                        lower="-2.09" upper="2.09" effort="500"
-                        velocity="3.14" damping="0.5"/>
-    <!-- joint7 -->
+                        lower="-2.09" upper="2.09" effort="200"
+                        velocity="3.14" damping="10.0" friction="0.1"
+                        soft_lower="-2.0027" soft_upper="2.0027" k_velocity="10"/>
+    <!-- joint7: ±174° hard, ±169° soft -->
     <xacro:revolute_joint jname="joint7" parent="link6" child="link7"
                         xyz="0 -0.126 0" rpy="1.5708 0 0" axis="0 0 1"
-                        lower="-3.05" upper="3.05" effort="500"
-                        velocity="3.14" damping="0.5"/>
+                        lower="-3.05" upper="3.05" effort="200"
+                        velocity="3.14" damping="10.0" friction="0.1"
+                        soft_lower="-2.9627" soft_upper="2.9627" k_velocity="10"/>
     <joint name="tools_joint" type="fixed">
         <origin xyz="0.0 0.0 0.0" rpy="0.0 0.0 0.0"/>

File: src/iiwa_description/urdf/macros.xacro (robot description, xacro)
@@ -27,5 +27,5 @@
     </xacro:macro>
     <!-- Макрос для описания соединений -->
-    <xacro:macro name="revolute_joint" params="jname parent child xyz rpy axis lower upper effort velocity damping">
+    <xacro:macro name="revolute_joint" params="jname parent child xyz rpy axis lower upper effort velocity damping friction soft_lower soft_upper k_velocity">
         <joint name="${jname}" type="revolute">
             <origin xyz="${xyz}" rpy="${rpy}"/>
@@ -34,5 +34,6 @@
             <axis xyz="${axis}"/>
             <limit lower="${lower}" upper="${upper}" effort="${effort}" velocity="${velocity}"/>
-            <dynamics damping="${damping}"/>
+            <dynamics damping="${damping}" friction="${friction}"/>
+            <safety_controller soft_lower_limit="${soft_lower}" soft_upper_limit="${soft_upper}" k_velocity="${k_velocity}"/>
         </joint>
     </xacro:macro>

File: src/iiwa_description/urdf/params.xacro (robot description, xacro)
@@ -2,5 +2,5 @@
 <robot xmlns:xacro="http://www.ros.org/wiki/xacro" xacro:version="1.0">
     <!-- Массы звеньев -->
-    <xacro:property name="mass_base" value="0.1"/>
+    <xacro:property name="mass_base" value="4.86"/>
     <xacro:property name="mass_link1" value="4"/>
     <xacro:property name="mass_link2" value="4"/>
