Commit message: Update camera settings

File: src/iiwa_description/urdf/iiwa7.urdf.xacro (robot description, xacro)
@@ -14,4 +14,5 @@
     <xacro:include filename="$(find iiwa_description)/urdf/links.xacro"/>
     <xacro:include filename="$(find iiwa_description)/urdf/joints.xacro"/>
+    <xacro:property name="tool_has_camera" value="false"/>
     <xacro:include filename="$(find iiwa_description)/urdf/tools/tool_active.xacro"/>
     <xacro:if value="$(arg simulate)">
@@ -20,4 +21,5 @@
             <device reference="camera_rgb" type="Camera">
                 <ros>
+                    <enabled>false</enabled>
                     <topicName>/camera/color</topicName>
                     <updateRate>30</updateRate>
@@ -28,4 +30,5 @@
             <device reference="camera_depth" type="RangeFinder">
                 <ros>
+                    <enabled>false</enabled>
                     <topicName>/camera/depth</topicName>
                     <updateRate>30</updateRate>
@@ -34,4 +37,20 @@
                 </ros>
             </device>
+            <!-- Keep the 30 Hz deadlines independent of Webots' 32 ms steps. -->
+            <xacro:if value="${tool_has_camera}">
+                <plugin type="iiwa_utils.webots_camera.WebotsCamera">
+                    <device>camera_rgb</device>
+                    <topicName>/camera/color</topicName>
+                    <updateRate>30</updateRate>
+                    <frameName>camera_optical_frame</frameName>
+                </plugin>
+                <plugin type="iiwa_utils.webots_camera.WebotsCamera">
+                    <device>camera_depth</device>
+                    <depth>true</depth>
+                    <topicName>/camera/depth</topicName>
+                    <updateRate>30</updateRate>
+                    <frameName>camera_optical_frame</frameName>
+                </plugin>
+            </xacro:if>
         </webots>
         <ros2_control name="iiwaGazeboControl" type="system">

File: src/iiwa_description/urdf/tools/patron.xacro (robot description, xacro)
@@ -1,4 +1,5 @@
 <?xml version="1.0"?>
 <robot xmlns:xacro="http://www.ros.org/wiki/xacro" name="tool_patron">
+    <xacro:property name="tool_has_camera" value="true"/>
     <link name="camera_holder">
         <inertial>
@@ -123,5 +124,6 @@
         <sensor type="camera" name="camera_rgb">
             <camera>
-                <horizontal_fov>1.3089969</horizontal_fov>
+                <!-- VGA RGB central-crop approximation: 79.61 deg; calibrate per device. -->
+                <horizontal_fov>1.3894765524</horizontal_fov>
                 <image>
                     <width>640</width>
@@ -135,5 +137,5 @@
                 <noise>
                     <type>gaussian</type>
-                    <stddev>0.005</stddev>
+                    <stddev>0.0</stddev>
                 </noise>
             </camera>
@@ -147,10 +149,11 @@
                 </image>
                 <clip>
-                    <near>0.52</near>
+                    <near>0.01</near>
                     <far>6.0</far>
                 </clip>
             </camera>
             <range>
-                <min>0.52</min>
+                <!-- Conservative simulation cutoff, not calibrated VGA Min-Z. -->
+                <min>0.4</min>
                 <max>6.0</max>
                 <resolution>0.001</resolution>
@@ -158,5 +161,6 @@
             <noise>
                 <type>gaussian</type>
-                <stddev>0.02</stddev>
+                <!-- No arbitrary Gaussian noise: this is an ideal depth model. -->
+                <stddev>0.0</stddev>
             </noise>
         </sensor>

Commit message: feat(control): unify joint limits and bound trajectory dynamics
Use shared limits for all seven axes across MoveIt, URDF and FRI.
Apply Ruckig smoothing and continuous JTC spline checks, stretching
trajectory timing to respect velocity, acceleration and jerk limits.
Require fresh stationary feedback for direct trajectories and protect
preparation from concurrent submissions and stop requests.

Add regression tests, dependencies and bilingual FRI documentation.
Include the updated LIN speed-sweep scenario and current 60 ms filter
configuration. Acceleration and jerk limits remain project settings;
physical high-speed twitching is still under investigation.

File: src/iiwa_description/urdf/iiwa7.urdf.xacro (robot description, xacro)
@@ -3,4 +3,6 @@
     <xacro:arg name="initial_positions_file"
                default="$(find iiwa_config)/config/moveit/initial_positions.yaml"/>
+    <xacro:arg name="joint_limits_file" default="$(find iiwa_config)/config/moveit/joint_limits.yaml"/>
+    <xacro:property name="joint_limits" value="${xacro.load_yaml('$(arg joint_limits_file)')['joint_limits']}"/>
     <xacro:arg name="simulate" default="false"/>
     <xacro:arg name="robot_ip" default="192.170.10.2"/>
@@ -41,6 +43,6 @@
             <joint name="joint1">
                 <command_interface name="position">
-                    <param name="min">-2.97</param>
-                    <param name="max"> 2.97</param>
+                    <param name="min">${joint_limits['joint1']['soft_min_position']}</param>
+                    <param name="max">${joint_limits['joint1']['soft_max_position']}</param>
                 </command_interface>
                 <state_interface name="position">
@@ -52,6 +54,6 @@
             <joint name="joint2">
                 <command_interface name="position">
-                    <param name="min">-2.09</param>
-                    <param name="max"> 2.09</param>
+                    <param name="min">${joint_limits['joint2']['soft_min_position']}</param>
+                    <param name="max">${joint_limits['joint2']['soft_max_position']}</param>
                 </command_interface>
                 <state_interface name="position">
@@ -63,6 +65,6 @@
             <joint name="joint3">
                 <command_interface name="position">
-                    <param name="min">-2.97</param>
-                    <param name="max"> 2.97</param>
+                    <param name="min">${joint_limits['joint3']['soft_min_position']}</param>
+                    <param name="max">${joint_limits['joint3']['soft_max_position']}</param>
                 </command_interface>
                 <state_interface name="position">
@@ -74,6 +76,6 @@
             <joint name="joint4">
                 <command_interface name="position">
-                    <param name="min">-2.09</param>
-                    <param name="max"> 2.09</param>
+                    <param name="min">${joint_limits['joint4']['soft_min_position']}</param>
+                    <param name="max">${joint_limits['joint4']['soft_max_position']}</param>
                 </command_interface>
                 <state_interface name="position">
@@ -85,6 +87,6 @@
             <joint name="joint5">
                 <command_interface name="position">
-                    <param name="min">-2.97</param>
-                    <param name="max"> 2.97</param>
+                    <param name="min">${joint_limits['joint5']['soft_min_position']}</param>
+                    <param name="max">${joint_limits['joint5']['soft_max_position']}</param>
                 </command_interface>
                 <state_interface name="position">
@@ -96,6 +98,6 @@
             <joint name="joint6">
                 <command_interface name="position">
-                    <param name="min">-2.09</param>
-                    <param name="max"> 2.09</param>
+                    <param name="min">${joint_limits['joint6']['soft_min_position']}</param>
+                    <param name="max">${joint_limits['joint6']['soft_max_position']}</param>
                 </command_interface>
                 <state_interface name="position">
@@ -107,6 +109,6 @@
             <joint name="joint7">
                 <command_interface name="position">
-                    <param name="min">-3.05</param>
-                    <param name="max"> 3.05</param>
+                    <param name="min">${joint_limits['joint7']['soft_min_position']}</param>
+                    <param name="max">${joint_limits['joint7']['soft_max_position']}</param>
                 </command_interface>
                 <state_interface name="position">
@@ -131,6 +133,6 @@
             <joint name="joint1">
                 <command_interface name="position">
-                    <param name="min">-2.97</param>
-                    <param name="max"> 2.97</param>
+                    <param name="min">${joint_limits['joint1']['soft_min_position']}</param>
+                    <param name="max">${joint_limits['joint1']['soft_max_position']}</param>
                 </command_interface>
                 <state_interface name="position">
@@ -142,6 +144,6 @@
             <joint name="joint2">
                 <command_interface name="position">
-                    <param name="min">-2.09</param>
-                    <param name="max"> 2.09</param>
+                    <param name="min">${joint_limits['joint2']['soft_min_position']}</param>
+                    <param name="max">${joint_limits['joint2']['soft_max_position']}</param>
                 </command_interface>
                 <state_interface name="position">
@@ -153,6 +155,6 @@
             <joint name="joint3">
                 <command_interface name="position">
-                    <param name="min">-2.97</param>
-                    <param name="max"> 2.97</param>
+                    <param name="min">${joint_limits['joint3']['soft_min_position']}</param>
+                    <param name="max">${joint_limits['joint3']['soft_max_position']}</param>
                 </command_interface>
                 <state_interface name="position">
@@ -164,6 +166,6 @@
             <joint name="joint4">
                 <command_interface name="position">
-                    <param name="min">-2.09</param>
-                    <param name="max"> 2.09</param>
+                    <param name="min">${joint_limits['joint4']['soft_min_position']}</param>
+                    <param name="max">${joint_limits['joint4']['soft_max_position']}</param>
                 </command_interface>
                 <state_interface name="position">
@@ -175,6 +177,6 @@
             <joint name="joint5">
                 <command_interface name="position">
-                    <param name="min">-2.97</param>
-                    <param name="max"> 2.97</param>
+                    <param name="min">${joint_limits['joint5']['soft_min_position']}</param>
+                    <param name="max">${joint_limits['joint5']['soft_max_position']}</param>
                 </command_interface>
                 <state_interface name="position">
@@ -186,6 +188,6 @@
             <joint name="joint6">
                 <command_interface name="position">
-                    <param name="min">-2.09</param>
-                    <param name="max"> 2.09</param>
+                    <param name="min">${joint_limits['joint6']['soft_min_position']}</param>
+                    <param name="max">${joint_limits['joint6']['soft_max_position']}</param>
                 </command_interface>
                 <state_interface name="position">
@@ -197,6 +199,6 @@
             <joint name="joint7">
                 <command_interface name="position">
-                    <param name="min">-3.05</param>
-                    <param name="max"> 3.05</param>
+                    <param name="min">${joint_limits['joint7']['soft_min_position']}</param>
+                    <param name="max">${joint_limits['joint7']['soft_max_position']}</param>
                 </command_interface>
                 <state_interface name="position">

File: src/iiwa_description/urdf/joints.xacro (robot description, xacro)
@@ -10,43 +10,43 @@
     <xacro:revolute_joint jname="joint1" parent="base_link" child="link1"
                         xyz="0 0 0.3375" rpy="0 0 0" axis="0 0 1"
-                        lower="-2.97" upper="2.97" effort="200"
-                        velocity="1.71" damping="10.0" friction="0.1"
-                        soft_lower="-2.8827" soft_upper="2.8827" k_velocity="10"/>
+                        lower="${joint_limits['joint1']['min_position']}" upper="${joint_limits['joint1']['max_position']}" effort="200"
+                        velocity="${joint_limits['joint1']['max_velocity']}" damping="10.0" friction="0.1"
+                        soft_lower="${joint_limits['joint1']['soft_min_position']}" soft_upper="${joint_limits['joint1']['soft_max_position']}" k_velocity="10"/>
     <!-- joint2: ±119° hard, ±114° soft -->
     <xacro:revolute_joint jname="joint2" parent="link1" child="link2"
                         xyz="0 0 0" rpy="-1.5708 0 0" axis="0 0 1"
-                        lower="-2.09" upper="2.09" effort="200"
-                        velocity="1.71" damping="10.0" friction="0.1"
-                        soft_lower="-2.0027" soft_upper="2.0027" k_velocity="10"/>
+                        lower="${joint_limits['joint2']['min_position']}" upper="${joint_limits['joint2']['max_position']}" effort="200"
+                        velocity="${joint_limits['joint2']['max_velocity']}" damping="10.0" friction="0.1"
+                        soft_lower="${joint_limits['joint2']['soft_min_position']}" soft_upper="${joint_limits['joint2']['soft_max_position']}" k_velocity="10"/>
     <!-- joint3: ±170° hard, ±165° soft -->
     <xacro:revolute_joint jname="joint3" parent="link2" child="link3"
                         xyz="0 -0.3993 0" rpy="1.5708 0 0" axis="0 0 1"
-                        lower="-2.97" upper="2.97" effort="200"
-                        velocity="1.75" damping="10.0" friction="0.1"
-                        soft_lower="-2.8827" soft_upper="2.8827" k_velocity="10"/>
+                        lower="${joint_limits['joint3']['min_position']}" upper="${joint_limits['joint3']['max_position']}" effort="200"
+                        velocity="${joint_limits['joint3']['max_velocity']}" damping="10.0" friction="0.1"
+                        soft_lower="${joint_limits['joint3']['soft_min_position']}" soft_upper="${joint_limits['joint3']['soft_max_position']}" k_velocity="10"/>
     <!-- joint4: ±119° hard, ±114° soft -->
     <xacro:revolute_joint jname="joint4" parent="link3" child="link4"
                         xyz="0 0 0" rpy="-1.5708 0 0" axis="0 0 -1"
-                        lower="-2.09" upper="2.09" effort="200"
-                        velocity="2.27" damping="10.0" friction="0.1"
-                        soft_lower="-2.0027" soft_upper="2.0027" k_velocity="10"/>
+                        lower="${joint_limits['joint4']['min_position']}" upper="${joint_limits['joint4']['max_position']}" effort="200"
+                        velocity="${joint_limits['joint4']['max_velocity']}" damping="10.0" friction="0.1"
+                        soft_lower="${joint_limits['joint4']['soft_min_position']}" soft_upper="${joint_limits['joint4']['soft_max_position']}" k_velocity="10"/>
     <!-- joint5: ±170° hard, ±165° soft -->
     <xacro:revolute_joint jname="joint5" parent="link4" child="link5"
                         xyz="0 -0.3993 0" rpy="1.5708 0 0" axis="0 0 1"
-                        lower="-2.97" upper="2.97" effort="200"
-                        velocity="2.44" damping="10.0" friction="0.1"
-                        soft_lower="-2.8827" soft_upper="2.8827" k_velocity="10"/>
+                        lower="${joint_limits['joint5']['min_position']}" upper="${joint_limits['joint5']['max_position']}" effort="200"
+                        velocity="${joint_limits['joint5']['max_velocity']}" damping="10.0" friction="0.1"
+                        soft_lower="${joint_limits['joint5']['soft_min_position']}" soft_upper="${joint_limits['joint5']['soft_max_position']}" k_velocity="10"/>
     <!-- joint6: ±119° hard, ±114° soft -->
     <xacro:revolute_joint jname="joint6" parent="link5" child="link6"
                         xyz="0 0 0" rpy="-1.5708 0 0" axis="0 0 1"
-                        lower="-2.09" upper="2.09" effort="200"
-                        velocity="3.14" damping="10.0" friction="0.1"
-                        soft_lower="-2.0027" soft_upper="2.0027" k_velocity="10"/>
+                        lower="${joint_limits['joint6']['min_position']}" upper="${joint_limits['joint6']['max_position']}" effort="200"
+                        velocity="${joint_limits['joint6']['max_velocity']}" damping="10.0" friction="0.1"
+                        soft_lower="${joint_limits['joint6']['soft_min_position']}" soft_upper="${joint_limits['joint6']['soft_max_position']}" k_velocity="10"/>
     <!-- joint7: ±174° hard, ±169° soft -->
     <xacro:revolute_joint jname="joint7" parent="link6" child="link7"
                         xyz="0 -0.126 0" rpy="1.5708 0 0" axis="0 0 1"
-                        lower="-3.05" upper="3.05" effort="200"
-                        velocity="3.14" damping="10.0" friction="0.1"
-                        soft_lower="-2.9627" soft_upper="2.9627" k_velocity="10"/>
+                        lower="${joint_limits['joint7']['min_position']}" upper="${joint_limits['joint7']['max_position']}" effort="200"
+                        velocity="${joint_limits['joint7']['max_velocity']}" damping="10.0" friction="0.1"
+                        soft_lower="${joint_limits['joint7']['soft_min_position']}" soft_upper="${joint_limits['joint7']['soft_max_position']}" k_velocity="10"/>
     <joint name="tools_joint" type="fixed">
         <origin xyz="0.0 0.0 0.0" rpy="0.0 0.0 0.0"/>
