Commit message: Refactor URDF and launch files for iiwa robot
- Updated gripper macros in gripper_macros.xacro to simplify parameters and add Gazebo support.
- Removed unused mesh property in gripper_meshes.xacro.
- Enhanced iiwa7 digital and FRI URDF files with simulation arguments and improved controller setup.
- Added new launch files for Gazebo simulation and universal launch configuration.
- Implemented YAML parameter wrapping for ROS2 in converter.py.
- Introduced a new gz_bridge.yaml configuration for Gazebo to ROS2 topic mapping.
- Cleaned up setting_loader.py and added necessary imports.

File: src/iiwa_description/urdf/gripper/___gripper.urdf (robot description, URDF)
Before this commit: robot gripper, 9 links, 8 joints
Links:
- removed link craving1
- removed link craving2
- removed link craving3
- link screw: geometry visual mesh filename=/home/daniel/dev/kuka_iiwa7_ros2/src/iiwa_description/resou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
Joints:
- removed joint craving1_joint
- removed joint craving2_joint
- removed joint craving3_joint
- joint base: origin xyz=0.0 0.0 61 rpy=0.0 0.0 0.0 -> xyz=0.0 0.0 61.3 rpy=0.0 0.0 0.0
- joint finger1_joint: limit lower=-0.2 upper=0.09 effort=0.0 velocity=0.0 -> lower=-0.2 upper=0.07 effort=0.0 velocity=0.0
- joint finger2_joint: limit lower=-0.2 upper=0.09 effort=0.0 velocity=0.0 -> lower=-0.2 upper=0.07 effort=0.0 velocity=0.0
- joint finger3_joint: limit lower=-0.2 upper=0.09 effort=0.0 velocity=0.0 -> lower=-0.2 upper=0.07 effort=0.0 velocity=0.0

File: src/iiwa_description/urdf/gripper/gripper.xacro (robot description, xacro)
@@ -1,11 +1,8 @@
 <?xml version="1.0"?>
-<!-- Захват для Webots digital twin: все суставы fixed, без физики суставов.
-     Для реального робота используй gripper.xacro. -->
 <robot xmlns:xacro="http://www.ros.org/wiki/xacro" xacro:version="1.0">
-    <!-- Digital: box collision вместо mesh, все суставы с правильной физикой -->
     <xacro:include filename="$(find iiwa_description)/urdf/gripper/gripper_links.xacro"/>
     <xacro:include filename="$(find iiwa_description)/urdf/gripper/gripper_joints.xacro"/>
     <joint name="gripper_attach_joint" type="fixed">
-        <origin xyz="0.0 0.0 0" rpy="0.0 0.0 0.0"/>
+        <origin xyz="0.0 0.0 0.0" rpy="0.0 0.0 0.0"/>
         <parent link="link_ee"/>
         <child link="base_frame"/>

File: src/iiwa_description/urdf/gripper/gripper_joints.xacro (robot description, xacro)
@@ -2,6 +2,7 @@
 <robot xmlns:xacro="http://www.ros.org/wiki/xacro" xacro:version="1.0">
     <xacro:include filename="$(find iiwa_description)/urdf/gripper/gripper_macros.xacro"/>
+    <xacro:arg name="simulate" default="false"/>
     <joint name="base_joint" type="fixed">
-        <origin xyz="0.0 0.0 0.061" rpy="0.0 0.0 0.0"/>
+        <origin xyz="0.0 0.0 0.0613" rpy="0.0 0.0 0.0"/>
         <parent link="base_frame"/>
         <child link="plate"/>
@@ -13,27 +14,9 @@
         lower="-0.007" upper="0.0"
         effort="50.0" velocity="0.05"/>
-    <xacro:mimic_revolute_joint jname="craving1_joint"
-        parent="screw" child="craving1"
-        xyz="0.0155 -0.0095 0.004" rpy="0.0 0 -0.55"
-        axis="0.0 1 0.0"
-        lower="-0.25" upper="-0.2" effort="5.0" velocity="1.0" damping="0.05"
-        mimic_joint="base_screw" multiplier="0.1" mimic_offset="-0.25"/>
-    <xacro:mimic_revolute_joint jname="craving2_joint"
-        parent="screw" child="craving2"
-        xyz="-0.0155 -0.0095 0.004" rpy="0.0 0 0.55"
-        axis="0.0 1 0.0"
-        lower="0.2" upper="0.25" effort="5.0" velocity="1.0" damping="0.05"
-        mimic_joint="base_screw" multiplier="0.1" mimic_offset="0.2"/>
-    <xacro:mimic_revolute_joint jname="craving3_joint"
-        parent="screw" child="craving3"
-        xyz="0 0.018 0.004" rpy="0.0 0 1.57"
-        axis="0.0 1 0.0"
-        lower="-0.25" upper="-0.2" effort="5.0" velocity="1.0" damping="0.05"
-        mimic_joint="base_screw" multiplier="0.1" mimic_offset="-0.25"/>
     <xacro:mimic_revolute_joint jname="finger1_joint"
         parent="plate" child="finger1"
         xyz="0.0315 -0.0185 0.028" rpy="0.0 0.0 -2.12"
         axis="1 0.0 0"
-        lower="-0.2" upper="0.09" effort="5.0" velocity="1.0" damping="0.0"
+        lower="-0.2" upper="0.07" effort="5.0" velocity="1.0" damping="0.0"
         mimic_joint="base_screw" multiplier="-50" mimic_offset="-0.2"/>
     <xacro:mimic_revolute_joint jname="finger2_joint"
@@ -41,5 +24,5 @@
         xyz="-0.0315 -0.0185 0.028" rpy="0.0 0.0 2.12"
         axis="1 0.0 0"
-        lower="-0.2" upper="0.09" effort="5.0" velocity="1.0" damping="0.0"
+        lower="-0.2" upper="0.07" effort="5.0" velocity="1.0" damping="0.0"
         mimic_joint="base_screw" multiplier="-50" mimic_offset="-0.2"/>
     <xacro:mimic_revolute_joint jname="finger3_joint"
@@ -47,5 +30,5 @@
         xyz="0 0.037 0.028" rpy="0.0 0.0 0.0"
         axis="1 0.0 0"
-        lower="-0.2" upper="0.09" effort="5.0" velocity="1.0" damping="0.0"
+        lower="-0.2" upper="0.07" effort="5.0" velocity="1.0" damping="0.0"
         mimic_joint="base_screw" multiplier="-50" mimic_offset="-0.2"/>
 </robot>

File: src/iiwa_description/urdf/gripper/gripper_links.xacro (robot description, xacro)
@@ -1,8 +1,5 @@
 <?xml version="1.0"?>
-<!-- Links захвата для Webots digital twin.
-     Использует gripper_macros_digital.xacro: visual=mesh, collision=box.
-     Размеры box определены по смещениям суставов и геометрии захвата. -->
 <robot xmlns:xacro="http://www.ros.org/wiki/xacro" xacro:version="1.0">
-    <xacro:include filename="$(find iiwa_description)/urdf/gripper/gripper_macros_digital.xacro"/>
+    <xacro:include filename="$(find iiwa_description)/urdf/gripper/gripper_macros.xacro"/>
     <xacro:include filename="$(find iiwa_description)/urdf/gripper/gripper_meshes.xacro"/>
     <xacro:property name="gripper_dark_r" value="0.05"/>
@@ -15,5 +12,4 @@
     <xacro:property name="gripper_finger_g" value="0.8"/>
     <xacro:property name="gripper_finger_b" value="1.0"/>
-    <!-- base_frame: основной корпус ~44×44×72mm -->
     <xacro:gripper_link name="base_frame"
         mass="0.3" xyz_iner="0 0 0.035"
@@ -22,7 +18,5 @@
         mesh="${mesh_gripper_base_frame}"
         visual_xyz="-0.021 -0.021 0.006" visual_rpy="0 0 0"
-        r="${gripper_dark_r}" g="${gripper_dark_g}" b="${gripper_dark_b}" a="1.0"
-        box_x="0.044" box_y="0.044" box_z="0.072" box_xyz="0 0 0.036"/>
-    <!-- plate: пластина ~70×70×10mm -->
+        r="${gripper_dark_r}" g="${gripper_dark_g}" b="${gripper_dark_b}" a="1.0"/>
     <xacro:gripper_link name="plate"
         mass="0.15" xyz_iner="0 0 0"
@@ -31,7 +25,5 @@
         mesh="${mesh_gripper_plate}"
         visual_xyz="0 0 0" visual_rpy="0 0 0"
-        r="${gripper_alum_r}" g="${gripper_alum_g}" b="${gripper_alum_b}" a="1.0"
-        box_x="0.070" box_y="0.070" box_z="0.012" box_xyz="0 0 0.006"/>
-    <!-- screw: ходовой винт ~20×20×15mm -->
+        r="${gripper_alum_r}" g="${gripper_alum_g}" b="${gripper_alum_b}" a="1.0"/>
     <xacro:gripper_link name="screw"
         mass="0.03" xyz_iner="0 0 0"
@@ -40,32 +32,5 @@
         mesh="${mesh_gripper_screw}"
         visual_xyz="0 0 0" visual_rpy="0 0 0"
-        r="${gripper_alum_r}" g="${gripper_alum_g}" b="${gripper_alum_b}" a="1.0"
-        box_x="0.020" box_y="0.020" box_z="0.015" box_xyz="0 0 0"/>
-    <!-- craving1/2/3: кулачки ~12×12×35mm -->
-    <xacro:gripper_link name="craving1"
-        mass="0.01" xyz_iner="0 0 0"
-        ixx="0.000008" ixy="0.0" ixz="0.0"
-        iyy="0.000008" iyz="0.0" izz="0.000004"
-        mesh="${mesh_gripper_craving}"
-        visual_xyz="-0.004 -0.007 0.019" visual_rpy="0 1.57 0"
-        r="${gripper_alum_r}" g="${gripper_alum_g}" b="${gripper_alum_b}" a="1.0"
-        box_x="0.012" box_y="0.012" box_z="0.035" box_xyz="0 0 0.017"/>
-    <xacro:gripper_link name="craving2"
-        mass="0.01" xyz_iner="0 0 0"
-        ixx="0.000008" ixy="0.0" ixz="0.0"
-        iyy="0.000008" iyz="0.0" izz="0.000004"
-        mesh="${mesh_gripper_craving}"
-        visual_xyz="-0.004 -0.007 0.019" visual_rpy="0 1.57 0"
-        r="${gripper_alum_r}" g="${gripper_alum_g}" b="${gripper_alum_b}" a="1.0"
-        box_x="0.012" box_y="0.012" box_z="0.035" box_xyz="0 0 0.017"/>
-    <xacro:gripper_link name="craving3"
-        mass="0.01" xyz_iner="0 0 0"
-        ixx="0.000008" ixy="0.0" ixz="0.0"
-        iyy="0.000008" iyz="0.0" izz="0.000004"
-        mesh="${mesh_gripper_craving}"
-        visual_xyz="-0.004 -0.007 0.019" visual_rpy="0 1.57 0"
-        r="${gripper_alum_r}" g="${gripper_alum_g}" b="${gripper_alum_b}" a="1.0"
-        box_x="0.012" box_y="0.012" box_z="0.035" box_xyz="0 0 0.017"/>
-    <!-- finger1/2/3: пальцы ~10×10×40mm -->
+        r="${gripper_alum_r}" g="${gripper_alum_g}" b="${gripper_alum_b}" a="1.0"/>
     <xacro:gripper_link name="finger1"
         mass="0.015" xyz_iner="0 0 0"
@@ -74,6 +39,5 @@
         mesh="${mesh_gripper_finger}"
         visual_xyz="0.009 -0.025 0.005" visual_rpy="0 -1.57 0"
-        r="${gripper_finger_r}" g="${gripper_finger_g}" b="${gripper_finger_b}" a="1.0"
-        box_x="0.010" box_y="0.010" box_z="0.040" box_xyz="0 0 0.020"/>
+        r="${gripper_finger_r}" g="${gripper_finger_g}" b="${gripper_finger_b}" a="1.0"/>
     <xacro:gripper_link name="finger2"
         mass="0.015" xyz_iner="0 0 0"
@@ -82,6 +46,5 @@
         mesh="${mesh_gripper_finger}"
         visual_xyz="0.009 -0.025 0.005" visual_rpy="0 -1.57 0"
-        r="${gripper_finger_r}" g="${gripper_finger_g}" b="${gripper_finger_b}" a="1.0"
-        box_x="0.010" box_y="0.010" box_z="0.040" box_xyz="0 0 0.020"/>
+        r="${gripper_finger_r}" g="${gripper_finger_g}" b="${gripper_finger_b}" a="1.0"/>
     <xacro:gripper_link name="finger3"
         mass="0.015" xyz_iner="0 0 0"
@@ -90,5 +53,4 @@
         mesh="${mesh_gripper_finger}"
         visual_xyz="0.009 -0.025 0.005" visual_rpy="0 -1.57 0"
-        r="${gripper_finger_r}" g="${gripper_finger_g}" b="${gripper_finger_b}" a="1.0"
-        box_x="0.010" box_y="0.010" box_z="0.040" box_xyz="0 0 0.020"/>
+        r="${gripper_finger_r}" g="${gripper_finger_g}" b="${gripper_finger_b}" a="1.0"/>
 </robot>

File: src/iiwa_description/urdf/gripper/gripper_macros.xacro (robot description, xacro)
@@ -4,8 +4,6 @@
                  params="name mass
                          ixx ixy ixz iyy iyz izz xyz_iner
-                         mesh
-                         visual_xyz visual_rpy
-                         r g b a
-                         box_x box_y box_z box_xyz">
+                         mesh visual_xyz visual_rpy
+                         r g b a">
         <link name="${name}">
             <inertial>
@@ -25,10 +23,29 @@
             </visual>
             <collision>
-                <origin xyz="${box_xyz}" rpy="0 0 0"/>
+                <origin xyz="${visual_xyz}" rpy="${visual_rpy}"/>
                 <geometry>
-                    <box size="${box_x} ${box_y} ${box_z}"/>
+                    <mesh filename="${mesh}" scale="0.001 0.001 0.001"/>
                 </geometry>
             </collision>
         </link>
+        <gazebo reference="${name}">
+            <visual>
+                <material>
+                    <ambient>${r} ${g} ${b} ${a}</ambient>
+                    <diffuse>${r} ${g} ${b} ${a}</diffuse>
+                    <specular>0.3 0.3 0.3 1.0</specular>
+                </material>
+            </visual>
+            <collision>
+                <surface>
+                    <friction>
+                        <ode><mu>1.0</mu><mu2>1.0</mu2></ode>
+                    </friction>
+                    <contact>
+                        <ode><kp>1000000.0</kp><kd>100.0</kd></ode>
+                    </contact>
+                </surface>
+            </collision>
+        </gazebo>
     </xacro:macro>
     <xacro:macro name="prismatic_joint"

File: src/iiwa_description/urdf/gripper/gripper_meshes.xacro (robot description, xacro)
@@ -6,5 +6,4 @@
     <xacro:property name="mesh_gripper_plate" value="${gripper_pkg}/plate.stl"/>
     <xacro:property name="mesh_gripper_screw" value="${gripper_pkg}/screw.stl"/>
-    <xacro:property name="mesh_gripper_craving" value="${gripper_pkg}/craving.stl"/>
     <xacro:property name="mesh_gripper_finger" value="${gripper_pkg}/finger_plates.stl"/>
 </robot>

File: src/iiwa_description/urdf/iiwa7_digital.urdf.xacro (robot description, xacro)
@@ -4,4 +4,9 @@
     <xacro:arg name="initial_positions_file"
                default="$(find iiwa_config)/config/moveit/initial_positions.yaml"/>
+    <xacro:arg name="simulate" default="false"/>
+    <!-- Аргументы только для реального робота -->
+    <xacro:arg name="robot_ip" default="192.170.10.2"/>
+    <xacro:arg name="fri_port" default="30200"/>
+    <xacro:arg name="command_mode" default="position"/>
     <xacro:property name="initial_positions"
                     value="${xacro.load_yaml('$(arg initial_positions_file)')['initial_positions']}"/>
@@ -11,19 +16,38 @@
     <xacro:include filename="$(find iiwa_description)/urdf/joints.xacro"/>
     <xacro:include filename="$(find iiwa_description)/urdf/gripper/gripper.xacro"/>
-    <webots>
+    <xacro:if value="$(arg simulate)">
+        <gazebo>
+            <plugin filename="gz_ros2_control-system"
+                    name="gz_ros2_control::GazeboSimROS2ControlPlugin">
+                <parameters>$(find iiwa_config)/config/moveit/iiwa_controller.yaml</parameters>
+                <ros>
+                    <remapping>~/robot_description:=/robot_description</remapping>
+                </ros>
+            </plugin>
+        </gazebo>
+    </xacro:if>
+    <!-- <webots>
         <plugin type="webots_ros2_control::Ros2Control"/>
-    </webots>
-    <ros2_control name="iiwaWebotsControl" type="system">
+    </webots> -->
+    <ros2_control name="iiwaControl" type="system">
+        <xacro:if value="$(arg simulate)">
+            <hardware>
+                <plugin>gz_ros2_control/GazeboSimSystem</plugin>
+            </hardware>
+        </xacro:if>
         <hardware>
+            <plugin>iiwa_controller/IIWAHardwareInterface</plugin>
+            <param name="robot_ip">$(arg robot_ip)</param>
+            <param name="fri_port">$(arg fri_port)</param>
+            <param name="simulate">$(arg simulate)</param>
+            <param name="command_mode">$(arg command_mode)</param>
+        </hardware>
+         <!-- <hardware>
             <plugin>webots_ros2_control::Ros2ControlSystem</plugin>
-        </hardware>
-       <joint name="joint1">
+        </hardware> -->
+        <joint name="joint1">
             <command_interface name="position">
                 <param name="min">-2.97</param>
                 <param name="max"> 2.97</param>
-            </command_interface>
-            <command_interface name="effort">
-                <param name="min">-320</param>
-                <param name="max"> 320</param>
             </command_interface>
             <state_interface name="position">
@@ -38,8 +62,4 @@
                 <param name="max"> 2.09</param>
             </command_interface>
-            <command_interface name="effort">
-                <param name="min">-320</param>
-                <param name="max"> 320</param>
-            </command_interface>
             <state_interface name="position">
                 <param name="initial_value">${initial_positions['joint2']}</param>
@@ -52,8 +72,4 @@
                 <param name="min">-2.97</param>
                 <param name="max"> 2.97</param>
-            </command_interface>
-            <command_interface name="effort">
-                <param name="min">-320</param>
-                <param name="max"> 320</param>
             </command_interface>
             <state_interface name="position">
@@ -68,8 +84,4 @@
                 <param name="max"> 2.09</param>
             </command_interface>
-            <command_interface name="effort">
-                <param name="min">-320</param>
-                <param name="max"> 320</param>
-            </command_interface>
             <state_interface name="position">
                 <param name="initial_value">${initial_positions['joint4']}</param>
@@ -82,8 +94,4 @@
                 <param name="min">-2.97</param>
                 <param name="max"> 2.97</param>
-            </command_interface>
-            <command_interface name="effort">
-                <param name="min">-320</param>
-                <param name="max"> 320</param>
             </command_interface>
             <state_interface name="position">
@@ -98,8 +106,4 @@
                 <param name="max"> 2.09</param>
             </command_interface>
-            <command_interface name="effort">
-                <param name="min">-320</param>
-                <param name="max"> 320</param>
-            </command_interface>
             <state_interface name="position">
                 <param name="initial_value">${initial_positions['joint6']}</param>
@@ -113,8 +117,4 @@
                 <param name="max"> 3.05</param>
             </command_interface>
-            <command_interface name="effort">
-                <param name="min">-320</param>
-                <param name="max"> 320</param>
-            </command_interface>
             <state_interface name="position">
                 <param name="initial_value">${initial_positions['joint7']}</param>
@@ -123,6 +123,5 @@
             <state_interface name="effort"/>
         </joint>
-        <!-- Захват -->
-        <!-- <joint name="base_screw">
+        <joint name="base_screw">
             <command_interface name="position"/>
             <state_interface name="position">
@@ -130,5 +129,5 @@
             </state_interface>
             <state_interface name="velocity"/>
-        </joint> -->
+        </joint>
     </ros2_control>
 </robot>
