Commit message: Refactor URDF and launch files for iiwa robot
- Updated gripper macros in gripper_macros.xacro to simplify parameters and add Gazebo support.
- Removed unused mesh property in gripper_meshes.xacro.
- Enhanced iiwa7 digital and FRI URDF files with simulation arguments and improved controller setup.
- Added new launch files for Gazebo simulation and universal launch configuration.
- Implemented YAML parameter wrapping for ROS2 in converter.py.
- Introduced a new gz_bridge.yaml configuration for Gazebo to ROS2 topic mapping.
- Cleaned up setting_loader.py and added necessary imports.

File: src/iiwa_description/urdf/iiwa7_fri.urdf.xacro (robot description, xacro)
@@ -3,7 +3,7 @@
     <xacro:arg name="initial_positions_file"
                default="$(find iiwa_config)/config/moveit/initial_positions.yaml"/>
+    <xacro:arg name="simulate" default="false"/>
     <xacro:arg name="robot_ip" default="192.170.10.2"/>
     <xacro:arg name="fri_port" default="30200"/>
-    <xacro:arg name="simulate" default="false"/>
     <xacro:arg name="command_mode" default="position"/>
     <xacro:property name="initial_positions"
@@ -14,117 +14,219 @@
     <xacro:include filename="$(find iiwa_description)/urdf/joints.xacro"/>
     <xacro:include filename="$(find iiwa_description)/urdf/gripper/gripper.xacro"/>
-    <ros2_control name="iiwaFRIControl" type="system">
-        <hardware>
-            <plugin>iiwa_controller/IIWAHardwareInterface</plugin>
-            <param name="robot_ip">$(arg robot_ip)</param>
-            <param name="fri_port">$(arg fri_port)</param>
-            <param name="simulate">$(arg simulate)</param>
-            <param name="command_mode">$(arg command_mode)</param>
-        </hardware>
-        <joint name="joint1">
-            <command_interface name="position">
-                <param name="min">-2.97</param>
-                <param name="max"> 2.97</param>
-            </command_interface>
-            <command_interface name="effort">
-                <param name="min">-320</param>
-                <param name="max"> 320</param>
-            </command_interface>
-            <state_interface name="position">
-                <param name="initial_value">${initial_positions['joint1']}</param>
-            </state_interface>
-            <state_interface name="velocity"/>
-            <state_interface name="effort"/>
-        </joint>
-        <joint name="joint2">
-            <command_interface name="position">
-                <param name="min">-2.09</param>
-                <param name="max"> 2.09</param>
-            </command_interface>
-            <command_interface name="effort">
-                <param name="min">-320</param>
-                <param name="max"> 320</param>
-            </command_interface>
-            <state_interface name="position">
-                <param name="initial_value">${initial_positions['joint2']}</param>
-            </state_interface>
-            <state_interface name="velocity"/>
-            <state_interface name="effort"/>
-        </joint>
-        <joint name="joint3">
-            <command_interface name="position">
-                <param name="min">-2.97</param>
-                <param name="max"> 2.97</param>
-            </command_interface>
-            <command_interface name="effort">
-                <param name="min">-320</param>
-                <param name="max"> 320</param>
-            </command_interface>
-            <state_interface name="position">
-                <param name="initial_value">${initial_positions['joint3']}</param>
-            </state_interface>
-            <state_interface name="velocity"/>
-            <state_interface name="effort"/>
-        </joint>
-        <joint name="joint4">
-            <command_interface name="position">
-                <param name="min">-2.09</param>
-                <param name="max"> 2.09</param>
-            </command_interface>
-            <command_interface name="effort">
-                <param name="min">-320</param>
-                <param name="max"> 320</param>
-            </command_interface>
-            <state_interface name="position">
-                <param name="initial_value">${initial_positions['joint4']}</param>
-            </state_interface>
-            <state_interface name="velocity"/>
-            <state_interface name="effort"/>
-        </joint>
-        <joint name="joint5">
-            <command_interface name="position">
-                <param name="min">-2.97</param>
-                <param name="max"> 2.97</param>
-            </command_interface>
-            <command_interface name="effort">
-                <param name="min">-320</param>
-                <param name="max"> 320</param>
-            </command_interface>
-            <state_interface name="position">
-                <param name="initial_value">${initial_positions['joint5']}</param>
-            </state_interface>
-            <state_interface name="velocity"/>
-            <state_interface name="effort"/>
-        </joint>
-        <joint name="joint6">
-            <command_interface name="position">
-                <param name="min">-2.09</param>
-                <param name="max"> 2.09</param>
-            </command_interface>
-            <command_interface name="effort">
-                <param name="min">-320</param>
-                <param name="max"> 320</param>
-            </command_interface>
-            <state_interface name="position">
-                <param name="initial_value">${initial_positions['joint6']}</param>
-            </state_interface>
-            <state_interface name="velocity"/>
-            <state_interface name="effort"/>
-        </joint>
-        <joint name="joint7">
-            <command_interface name="position">
-                <param name="min">-3.05</param>
-                <param name="max"> 3.05</param>
-            </command_interface>
-            <command_interface name="effort">
-                <param name="min">-320</param>
-                <param name="max"> 320</param>
-            </command_interface>
-            <state_interface name="position">
-                <param name="initial_value">${initial_positions['joint7']}</param>
-            </state_interface>
-            <state_interface name="velocity"/>
-            <state_interface name="effort"/>
-        </joint>
-    </ros2_control>
+    <xacro:if value="$(arg simulate)">
+        <gazebo>
+            <plugin filename="gz_ros2_control-system"
+                    name="gz_ros2_control::GazeboSimROS2ControlPlugin">
+                <parameters>$(find iiwa_config)/config/moveit/iiwa_controller.yaml</parameters>
+                <ros>
+                    <remapping>~/robot_description:=/robot_description</remapping>
+                </ros>
+            </plugin>
+        </gazebo>
+        <ros2_control name="iiwaGazeboControl" type="system">
+            <hardware>
+                <plugin>gz_ros2_control/GazeboSimSystem</plugin>
+            </hardware>
+            <joint name="joint1">
+                <command_interface name="position">
+                    <param name="min">-2.97</param>
+                    <param name="max"> 2.97</param>
+                </command_interface>
+                <state_interface name="position">
+                    <param name="initial_value">${initial_positions['joint1']}</param>
+                </state_interface>
+                <state_interface name="velocity"/>
+                <state_interface name="effort"/>
+            </joint>
+            <joint name="joint2">
+                <command_interface name="position">
+                    <param name="min">-2.09</param>
+                    <param name="max"> 2.09</param>
+                </command_interface>
+                <state_interface name="position">
+                    <param name="initial_value">${initial_positions['joint2']}</param>
+                </state_interface>
+                <state_interface name="velocity"/>
+                <state_interface name="effort"/>
+            </joint>
+            <joint name="joint3">
+                <command_interface name="position">
+                    <param name="min">-2.97</param>
+                    <param name="max"> 2.97</param>
+                </command_interface>
+                <state_interface name="position">
+                    <param name="initial_value">${initial_positions['joint3']}</param>
+                </state_interface>
+                <state_interface name="velocity"/>
+                <state_interface name="effort"/>
+            </joint>
+            <joint name="joint4">
+                <command_interface name="position">
+                    <param name="min">-2.09</param>
+                    <param name="max"> 2.09</param>
+                </command_interface>
+                <state_interface name="position">
+                    <param name="initial_value">${initial_positions['joint4']}</param>
+                </state_interface>
+                <state_interface name="velocity"/>
+                <state_interface name="effort"/>
+            </joint>
+            <joint name="joint5">
+                <command_interface name="position">
+                    <param name="min">-2.97</param>
+                    <param name="max"> 2.97</param>
+                </command_interface>
+                <state_interface name="position">
+                    <param name="initial_value">${initial_positions['joint5']}</param>
+                </state_interface>
+                <state_interface name="velocity"/>
+                <state_interface name="effort"/>
+            </joint>
+            <joint name="joint6">
+                <command_interface name="position">
+                    <param name="min">-2.09</param>
+                    <param name="max"> 2.09</param>
+                </command_interface>
+                <state_interface name="position">
+                    <param name="initial_value">${initial_positions['joint6']}</param>
+                </state_interface>
+                <state_interface name="velocity"/>
+                <state_interface name="effort"/>
+            </joint>
+            <joint name="joint7">
+                <command_interface name="position">
+                    <param name="min">-3.05</param>
+                    <param name="max"> 3.05</param>
+                </command_interface>
+                <state_interface name="position">
+                    <param name="initial_value">${initial_positions['joint7']}</param>
+                </state_interface>
+                <state_interface name="velocity"/>
+                <state_interface name="effort"/>
+            </joint>
+            <joint name="base_screw">
+                <command_interface name="position"/>
+                <state_interface name="position">
+                    <param name="initial_value">0.0</param>
+                </state_interface>
+                <state_interface name="velocity"/>
+            </joint>
+        </ros2_control>
+    </xacro:if>
+    <xacro:unless value="$(arg simulate)">
+        <ros2_control name="iiwaFRIControl" type="system">
+            <hardware>
+                <plugin>iiwa_controller/IIWAHardwareInterface</plugin>
+                <param name="robot_ip">$(arg robot_ip)</param>
+                <param name="fri_port">$(arg fri_port)</param>
+                <param name="simulate">false</param>
+                <param name="command_mode">$(arg command_mode)</param>
+            </hardware>
+            <joint name="joint1">
+                <command_interface name="position">
+                    <param name="min">-2.97</param>
+                    <param name="max"> 2.97</param>
+                </command_interface>
+                <command_interface name="effort">
+                    <param name="min">-320</param>
+                    <param name="max"> 320</param>
+                </command_interface>
+                <state_interface name="position">
+                    <param name="initial_value">${initial_positions['joint1']}</param>
+                </state_interface>
+                <state_interface name="velocity"/>
+                <state_interface name="effort"/>
+            </joint>
+            <joint name="joint2">
+                <command_interface name="position">
+                    <param name="min">-2.09</param>
+                    <param name="max"> 2.09</param>
+                </command_interface>
+                <command_interface name="effort">
+                    <param name="min">-320</param>
+                    <param name="max"> 320</param>
+                </command_interface>
+                <state_interface name="position">
+                    <param name="initial_value">${initial_positions['joint2']}</param>
+                </state_interface>
+                <state_interface name="velocity"/>
+                <state_interface name="effort"/>
+            </joint>
+            <joint name="joint3">
+                <command_interface name="position">
+                    <param name="min">-2.97</param>
+                    <param name="max"> 2.97</param>
+                </command_interface>
+                <command_interface name="effort">
+                    <param name="min">-320</param>
+                    <param name="max"> 320</param>
+                </command_interface>
+                <state_interface name="position">
+                    <param name="initial_value">${initial_positions['joint3']}</param>
+                </state_interface>
+                <state_interface name="velocity"/>
+                <state_interface name="effort"/>
+            </joint>
+            <joint name="joint4">
+                <command_interface name="position">
+                    <param name="min">-2.09</param>
+                    <param name="max"> 2.09</param>
+                </command_interface>
+                <command_interface name="effort">
+                    <param name="min">-320</param>
+                    <param name="max"> 320</param>
+                </command_interface>
+                <state_interface name="position">
+                    <param name="initial_value">${initial_positions['joint4']}</param>
+                </state_interface>
+                <state_interface name="velocity"/>
+                <state_interface name="effort"/>
+            </joint>
+            <joint name="joint5">
+                <command_interface name="position">
+                    <param name="min">-2.97</param>
+                    <param name="max"> 2.97</param>
+                </command_interface>
+                <command_interface name="effort">
+                    <param name="min">-320</param>
+                    <param name="max"> 320</param>
+                </command_interface>
+                <state_interface name="position">
+                    <param name="initial_value">${initial_positions['joint5']}</param>
+                </state_interface>
+                <state_interface name="velocity"/>
+                <state_interface name="effort"/>
+            </joint>
+            <joint name="joint6">
+                <command_interface name="position">
+                    <param name="min">-2.09</param>
+                    <param name="max"> 2.09</param>
+                </command_interface>
+                <command_interface name="effort">
+                    <param name="min">-320</param>
+                    <param name="max"> 320</param>
+                </command_interface>
+                <state_interface name="position">
+                    <param name="initial_value">${initial_positions['joint6']}</param>
+                </state_interface>
+                <state_interface name="velocity"/>
+                <state_interface name="effort"/>
+            </joint>
+            <joint name="joint7">
+                <command_interface name="position">
+                    <param name="min">-3.05</param>
+                    <param name="max"> 3.05</param>
+                </command_interface>
+                <command_interface name="effort">
+                    <param name="min">-320</param>
+                    <param name="max"> 320</param>
+                </command_interface>
+                <state_interface name="position">
+                    <param name="initial_value">${initial_positions['joint7']}</param>
+                </state_interface>
+                <state_interface name="velocity"/>
+                <state_interface name="effort"/>
+            </joint>
+        </ros2_control>
+    </xacro:unless>
 </robot>

File: src/iiwa_description/urdf/macros.xacro (robot description, xacro)
@@ -25,4 +25,14 @@
             </collision>
         </link>
+        <gazebo reference="${name}">
+            <visual>
+                <material>
+                    <ambient>${color_r * 0.7} ${color_g * 0.7} ${color_b * 0.7} ${color_a}</ambient>
+                    <diffuse>${color_r} ${color_g} ${color_b} ${color_a}</diffuse>
+                    <specular>0.3 0.3 0.3 1.0</specular>
+                    <emissive>0 0 0 1</emissive>
+                </material>
+            </visual>
+        </gazebo>
     </xacro:macro>
     <!-- Макрос для описания соединений -->
