Commit message: Refactor controller launch configuration and remove deprecated URDF files

File: src/iiwa_description/urdf/gripper/gripper_macros.xacro (robot description, xacro)
@@ -29,23 +29,4 @@
             </collision>
         </link>
-        <gazebo reference="${name}">
-            <visual>
-                <material>
-                    <ambient>${r} ${g} ${b} ${a}</ambient>
-                    <diffuse>${r} ${g} ${b} ${a}</diffuse>
-                    <specular>0.3 0.3 0.3 1.0</specular>
-                </material>
-            </visual>
-            <collision>
-                <surface>
-                    <friction>
-                        <ode><mu>1.0</mu><mu2>1.0</mu2></ode>
-                    </friction>
-                    <contact>
-                        <ode><kp>1000000.0</kp><kd>100.0</kd></ode>
-                    </contact>
-                </surface>
-            </collision>
-        </gazebo>
     </xacro:macro>
     <xacro:macro name="prismatic_joint"

File: src/iiwa_description/urdf/macros.xacro (robot description, xacro)
@@ -25,14 +25,4 @@
             </collision>
         </link>
-        <gazebo reference="${name}">
-            <visual>
-                <material>
-                    <ambient>${color_r * 0.7} ${color_g * 0.7} ${color_b * 0.7} ${color_a}</ambient>
-                    <diffuse>${color_r} ${color_g} ${color_b} ${color_a}</diffuse>
-                    <specular>0.3 0.3 0.3 1.0</specular>
-                    <emissive>0 0 0 1</emissive>
-                </material>
-            </visual>
-        </gazebo>
     </xacro:macro>
     <!-- Макрос для описания соединений -->
