Commit message: feat: Enhance iiwa_description and iiwa_sunrise functionality
- Added a new link "tcp" and a fixed joint "patron_tcp" in patron.xacro for better tool control.
- Updated ServerFriRos2.java to improve command mode handling and user configuration steps, including clearer logging and better control mode selection.
- Removed the deprecated iiwa_ros2.java file to streamline the codebase.
- Enhanced test_motion_sequence.py to allow dynamic topic recording based on user input, with improved logging for bag file management.

File: src/iiwa_description/urdf/tools/patron.xacro (robot description, xacro)
@@ -88,4 +88,5 @@
     </link>
     <link name="camera_optical_frame"/>
+    <link name="tcp" />
     <joint name="tool" type="fixed">
         <parent link="link_ee"/>
@@ -97,4 +98,9 @@
         <parent link="camera_holder"/>
         <child link="patron"/>
+    </joint>
+    <joint name="patron_tcp" type="fixed">
+        <origin xyz="0.0 0.0 0.0" rpy="0.0 0.0 -1.5708"/>
+        <parent link="patron"/>
+        <child link="tcp"/>
     </joint>
     <joint name="camera_holder_corner" type="fixed">
